Commit message: zikki

File: urdf/er.urdf.xacro (robot description, xacro)
@@ -24,5 +24,5 @@
         <parent link="base_link"/>
         <child link="lidar_link"/>
-        <origin xyz="-0.3155 0 0" rpy="3.14 0 3.14"/>
+        <origin xyz="0 -0.3155 0" rpy="3.14 0 -1.57"/>
     </joint>
 </robot>

Commit message: succeed

File: urdf/er.urdf.xacro (robot description, xacro)
@@ -1,8 +1,8 @@
 <?xml version="1.0"?>
-<robot name="nav_omni4" xmlns:xacro="http://ros.org/wiki/xacro">
+<robot name="nav_omni4">
     <link name="base_link">
         <visual>
             <geometry>
-                <box size="0.14 0.14 0.015"/>
+                <box size="0.555 0.555 0.015"/>
             </geometry>
         </visual>
@@ -24,23 +24,5 @@
         <parent link="base_link"/>
         <child link="lidar_link"/>
-        <origin xyz="0 0 0.06" rpy="0 0 0"/>
-    </joint>
-    <link name="camera_link">
-        <visual>
-            <geometry>
-                <box size="0.01 0.015 0.01"/>
-            </geometry>
-        </visual>
-    </link>
-    <link name="camera_depth_frame"/>
-    <joint name="camera_depth_joint" type="fixed">
-		<origin xyz="0 0 0" rpy="-${pi/2} 0 -${pi/2}"/>
-        <parent link="camera_link"/>
-        <child link="camera_depth_frame"/>
-    </joint>
-    <joint name="camera_joint" type="fixed">
-        <parent link="base_link"/>
-        <child link="camera_link"/>
-        <origin xyz="0.07 0 0.05" rpy="0 0 0"/>
+        <origin xyz="0 -0.3155 0" rpy="3.14 0 -1.57"/>
     </joint>
 </robot>
